Commit message: Teleoperación de stubbs añadida.

File: stubbs_description/urdf/stubbs.xacro (robot description, xacro)
@@ -8,4 +8,5 @@
 <xacro:property name="body_length" value=".5"/>
 <xacro:property name="wheel_length" value=".05"/>
+<xacro:property name="wheel_radius" value=".1"/>
 <xacro:property name="caster_radius" value="0.025"/>
 <xacro:property name="body_mass" value="1"/>
@@ -41,11 +42,21 @@
 		<origin xyz="0 0 0" rpy="1.5707 0 0"/>
 		<geometry>
-			<cylinder length="${wheel_length}" radius=".1"/>
+			<cylinder length="${wheel_length}" radius="${wheel_radius}"/>
 		</geometry>
+		<surface>
+			<friction>
+				<ode>
+					<mu>100000.0</mu>
+					<mu2>100000.0</mu2>
+					<slip1>0.0</slip1>
+					<slip2>0.0</slip2>
+				</ode>
+			</friction>
+        </surface>
 	</collision>
 	<visual>
 		<origin xyz="0 0 0" rpy="1.5707 0 0"/>
 		<geometry>
-			<cylinder length="${wheel_length}" radius=".1"/>
+			<cylinder length="${wheel_length}" radius="${wheel_radius}"/>
 		</geometry>
 	</visual>
@@ -53,5 +64,5 @@
 		<origin xyz="0 0 0" rpy="0 0 0"/>
 		<mass value="${wheel_mass}"/>
-		<cylinder_inertia m="${wheel_mass}" r=".1" h="${wheel_length}"/>
+		<cylinder_inertia m="${wheel_mass}" r="${wheel_radius}" h="${wheel_length}"/>
 	</inertial>
 </link>
@@ -60,11 +71,21 @@
 		<origin xyz="0 0 0" rpy="1.5707 0 0"/>
 		<geometry>
-			<cylinder length="${wheel_length}" radius=".1"/>
+			<cylinder length="${wheel_length}" radius="${wheel_radius}"/>
 		</geometry>
+		<surface>
+			<friction>
+				<ode>
+					<mu>100000.0</mu>
+					<mu2>100000.0</mu2>
+					<slip1>0.0</slip1>
+					<slip2>0.0</slip2>
+				</ode>
+			</friction>
+        </surface>
 	</collision>
 	<visual>
 		<origin xyz="0 0 0" rpy="1.5707 0 0"/>
 		<geometry>
-			<cylinder length="${wheel_length}" radius=".1"/>
+			<cylinder length="${wheel_length}" radius="${wheel_radius}"/>
 		</geometry>
 	</visual>
@@ -72,5 +93,5 @@
 		<origin xyz="0 0 0" rpy="0 0 0"/>
 		<mass value="${wheel_mass}"/>
-		<cylinder_inertia m="${wheel_mass}" r=".1" h="${wheel_length}"/>
+		<cylinder_inertia m="${wheel_mass}" r="${wheel_radius}" h="${wheel_length}"/>
 	</inertial>
 </link>
@@ -99,5 +120,5 @@
 	<parent link="body"/>
 	<axis xyz="0 1 0"/>
-	<limit effort="100" velocity="100"/>
+	<limit effort="100" velocity="10"/>
 	<joint_properties damping="0.0" friction="0.0"/>
 </joint>
@@ -107,5 +128,5 @@
 	<parent link="body"/>
 	<axis xyz="0 1 0"/>
-	<limit effort="100" velocity="100"/>
+	<limit effort="100" velocity="10"/>
 	<joint_properties damping="0.0" friction="0.0"/>
 </joint>
@@ -122,5 +143,6 @@
 	</joint>
 	<actuator name="l_motor">
-		<mechanicalReduction>1</mechanicalReduction>
+		<hardwareInterface>EffortJointInterface</hardwareInterface>
+		<mechanicalReduction>10</mechanicalReduction>
 	</actuator>
 </transmission>
@@ -131,5 +153,6 @@
 	</joint>
 	<actuator name="r_motor">
-		<mechanicalReduction>1</mechanicalReduction>
+		<hardwareInterface>EffortJointInterface</hardwareInterface>
+		<mechanicalReduction>10</mechanicalReduction>
 	</actuator>
 </transmission>
